File: seismometer.sch (KiCad schematic (older format))
At the start: 27 parts, among them U1 LM7809CT, U2 LM7909CT, U3 TL081, U4 TL081, U5 TL081

Commit message: Schematic first draw
Parts:
- removed C?: C, ~, symbol C
- removed D7: DIODE, ~, symbol DIODE
- removed D8: ZENER, ~, symbol ZENER
- removed R1, R2, R3, R4, R5, R6: R, ~, symbol R
- removed U3, U4, U5: TL081, symbol TL081
- added C?: C, ~, symbol C
- added D? (x2): DIODE, ~, symbol DIODE
- added R? (x3): R, ~, symbol R
- added U?: TL081, symbol TL081
Connections:
- wire segments 99 -> 48

Commit message: Some changes. A.C.
Parts:
- added C? (x4): C, symbol C
- added R? (x13): R, symbol R
- added U? (x5): LM741, symbol LM741
Connections:
- wire segments 48 -> 101
Other:
- note added: "-(Vin)"
- note added: "A single channel"
- note added: "Adding offset."
- note added: "BLACK BOX \nbecause I didn't find the \ncomponent (charge pump)"
- note added: "Buffer. Input \nprotection \nmissing."
- note added: "Gain. Switchable gain? Various problems.\n"
- note added: "Low-pass"
- note added: "Offset. It could be common to all the channels."
- note added: "Old version, stand alone, not a shield. Delete it? Another project?"
- note added: "Vee with charge pump."
- note added: "Vin"
- moved on the sheet: C1, C2, C3, C4, C?, D1, D2, D3, D4, D5, D6, D?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
